File: mii_pcb_v0.kicad_pcb (KiCad board)
At the start: 2 copper layers, 8 parts, among them J1 CONN_02X05, J2 CONN_COAXIAL, J3 CONN_01X03, J4 CONN_01X03, J5 CONN_01X03, U1 WeMos_mini, U2 RFM69HW, U3 RFM69HCW

Commit message: new pcb
Parts:
- moved J2 73.9 mm to (206.4, 112.0)
- moved J1 59.3 mm to (207.8, 103.4), turned to 180 degrees
- moved U2 48.2 mm to (190.0, 104.2)
- moved J3 39.2 mm to (172.0, 97.6), turned to 90 degrees
- moved J4 35.9 mm to (172.0, 106.6), turned to 90 degrees
- moved U3 32.3 mm to (185.4, 104.2), turned to 180 degrees
- moved J5 29.2 mm to (172.0, 115.6), turned to 90 degrees
Routing:
- net /3.3V: track 0.00 -> 92.8 mm, vias 0 -> 3
- net /MISO: track 0.00 -> 52.2 mm, vias 0 -> 3
- net /MOSI: track 0.00 -> 44.6 mm, vias 0 -> 3
- net /SCK: track 0.00 -> 42.3 mm, vias 0 -> 1
- net /ANT: track 0.00 -> 41.8 mm, vias 0 -> 3
- net /A0: track 0.00 -> 37.8 mm, vias 0 -> 4
- net /SDA: track 0.00 -> 31.8 mm
- net /SCL: track 0.00 -> 31.5 mm
- net /NSS: track 0.00 -> 30.7 mm, vias 0 -> 2
- net /RX: track 0.00 -> 24.9 mm
- net /TX: track 0.00 -> 23.4 mm
- net /FLASH: track 0.00 -> 22.8 mm
- net /IRQ: track 0.00 -> 18.0 mm, vias 0 -> 2
- net /BTN: track 0.00 -> 11.9 mm
- net /GND: vias 0 -> 1
- added copper zone on B.Cu, net /GND
- added copper zone on F.Cu, net /GND
Other:
- board outline added: 42.4 x 27 mm
- board text added: "3.3"
- board text added: "5V"
- board text added: "A0"
- board text added: "ANT"
- board text added: "Antenna"
- board text added: "D0"
- board text added: "D1"
- board text added: "D2"
- board text added: "D3"
- board text added: "D4"
- board text added: "D5"
- board text added: "D6"
- board text added: "D7"
- board text added: "D8"
- board text added: "DIO0"
- board text added: "GND"
- board text added: "MISO"
- board text added: "MOSI"
- board text added: "NSS"
- board text added: "RFM69HCW"
- board text added: "RFM69HW"
- board text added: "RST"
- board text added: "RX"
- board text added: "SCK"
- board text added: "SCL"
- board text added: "SDA"
- board text added: "TX"
- board text added: "UEXT"

Commit message: Add jumper for Deepsleep
Parts:
- added JP1: Jumper, Pin_Headers:Pin_Header_Straight_1x02_Pitch2.54mm, F.Cu at (201.9, 92.7)
Connections:
- U1 pad 9: Net-(U1-Pad9) -> /RST
Routing:
- net /RST: track 0.00 -> 3.81 mm
- net /NSS: track 30.7 -> 34.1 mm
- net /MISO: track 52.2 -> 52.9 mm
Other:
- board text added: "DS"
